File: calcwriter_pins/calcwriter_pins.kicad_pcb (KiCad board)
At the start: 4 copper layers, 72 x 109 mm, 37 parts, among them J1 0965-0-15-20-80-14-11-0, J10 0965-0-15-20-80-14-11-0, J11 0965-0-15-20-80-14-11-0, J12 0965-0-15-20-80-14-11-0, J13 0965-0-15-20-80-14-11-0, J14 0965-0-15-20-80-14-11-0, J15 0965-0-15-20-80-14-11-0, J16 0965-0-15-20-80-14-11-0, J17 0965-0-15-20-80-14-11-0, J18 0965-0-15-20-80-14-11-0, J19 0965-0-15-20-80-14-11-0, J2 0965-0-15-20-80-14-11-0, J20 0965-0-15-20-80-14-11-0, J21 0965-0-15-20-80-14-11-0, J22 0965-0-15-20-80-14-11-0, J23 0965-0-15-20-80-14-11-0, J24 0965-0-15-20-80-14-11-0, J25 0965-0-15-20-80-14-11-0, J26 0965-0-15-20-80-14-11-0, J27 0965-0-15-20-80-14-11-0, J28 0965-0-15-20-80-14-11-0, J29 0965-0-15-20-80-14-11-0, J3 0965-0-15-20-80-14-11-0, J30 0965-0-15-20-80-14-11-0, J31 0965-0-15-20-80-14-11-0, J4 0965-0-15-20-80-14-11-0, J5 0965-0-15-20-80-14-11-0, J6 0965-0-15-20-80-14-11-0, J7 0965-0-15-20-80-14-11-0, J8 0965-0-15-20-80-14-11-0, J9 0965-0-15-20-80-14-11-0, P1 FH12-40S-0.5SH_55_

Commit message: did another thing AAAAAAAAAAAAAAAAAAA
Parts:
- removed CALC+2, CALC-2, J1, J10, J11, J12, J13, J14, J15, J16, J17, J18, J19, J2, J20, J21, J22, J23, J24, J25, J26, J27, J28, J29, J3, J30, J31, J4, J5, J6, J7, J8, J9: 0965-0-15-20-80-14-11-0, 0965-0-15-20-80-14-11-0:MILLMAX_0965-0-15-20-80-14-11-0
- removed the SCREW1 at (98.2, 52.5)
- removed SCREW2: MountingHole_2.2mm_M2, MountingHole:MountingHole_2.2mm_M2
- added A0: 0965-0-15-20-80-14-11-0, pogopin_smd:YZR0156-20033-02, B.Cu at (85.6, 71.7)
- added A1: 0965-0-15-20-80-14-11-0, pogopin_smd:YZR0156-20033-02, B.Cu at (84.1, 78.1)
- added A2: 0965-0-15-20-80-14-11-0, pogopin_smd:YZR0156-20033-02, B.Cu at (87.1, 81.1)
- added A3: 0965-0-15-20-80-14-11-0, pogopin_smd:YZR0156-20033-02, B.Cu at (90.7, 74.4)
- added A4: 0965-0-15-20-80-14-11-0, pogopin_smd:YZR0156-20033-02, B.Cu at (111.2, 142.0)
- added A5: 0965-0-15-20-80-14-11-0, pogopin_smd:YZR0156-20033-02, B.Cu at (116.0, 136.9)
- added A6: 0965-0-15-20-80-14-11-0, pogopin_smd:YZR0156-20033-02, B.Cu at (127.0, 129.9)
- added A7: 0965-0-15-20-80-14-11-0, pogopin_smd:YZR0156-20033-02, B.Cu at (95.1, 74.4)
- added B0: 0965-0-15-20-80-14-11-0, pogopin_smd:YZR0156-20033-02, B.Cu at (72.3, 74.6)
- added B1: 0965-0-15-20-80-14-11-0, pogopin_smd:YZR0156-20033-02, B.Cu at (71.1, 77.4)
- added B2: 0965-0-15-20-80-14-11-0, pogopin_smd:YZR0156-20033-02, B.Cu at (99.0, 78.0)
- added B3: 0965-0-15-20-80-14-11-0, pogopin_smd:YZR0156-20033-02, B.Cu at (98.3, 83.0)
- added B4: 0965-0-15-20-80-14-11-0, pogopin_smd:YZR0156-20033-02, B.Cu at (99.0, 90.1)
- added B5: 0965-0-15-20-80-14-11-0, pogopin_smd:YZR0156-20033-02, B.Cu at (99.3, 94.1)
- added B6: 0965-0-15-20-80-14-11-0, pogopin_smd:YZR0156-20033-02, B.Cu at (79.1, 130.6)
- added B7: 0965-0-15-20-80-14-11-0, pogopin_smd:YZR0156-20033-02, B.Cu at (86.6, 133.3)
- added CALC_NEG1: 0965-0-15-20-80-14-11-0, pogopin_smd:YZR0156-20033-02, B.Cu at (134.7, 66.2)
- added CALC_POS1: 0965-0-15-20-80-14-11-0, pogopin_smd:YZR0156-20033-02, B.Cu at (72.6, 63.0)
- added G***: LOGO, LOGO, F.Cu at (113.5, 124.8)
- added G***: LOGO, LOGO, F.Cu at (115.0, 75.2)
- added SCREW1: MountingHole_2.2mm_M2, MountingHole:MountingHole_2.2mm_M2, F.Cu at (92.5, 60.2)
- added SCREW1: MountingHole_2.2mm_M2, MountingHole:MountingHole_2.2mm_M2, F.Cu at (92.5, 84.8)
- moved ISP_HEADER1 21.8 mm to (102.8, 61.2)
- moved P1 18.0 mm to (81.0, 102.2)
Connections:
- P1 pad 10: /P24 -> unconnected-(P1-Pad10)
- P1 pad 11: /P23 -> unconnected-(P1-Pad11)
- P1 pad 12: /P22 -> unconnected-(P1-Pad12)
- P1 pad 13: /P21 -> unconnected-(P1-Pad13)
- P1 pad 14: /P20 -> unconnected-(P1-Pad14)
- P1 pad 15: /P19 -> unconnected-(P1-Pad15)
- P1 pad 16: /P18 -> unconnected-(P1-Pad16)
- P1 pad 17: /P17 -> unconnected-(P1-Pad17)
- P1 pad 18: /P16 -> +1V5
- P1 pad 19: /P15 -> /ISP_RST
- P1 pad 20: /P14 -> /ISP_SCK
- P1 pad 21: /P13 -> /ISP_MOSI
- P1 pad 22: /P12 -> /ISP_MISO
- P1 pad 23: /P11 -> /B3
- P1 pad 24: /P10 -> /B0
- P1 pad 25: /P9 -> /B1
- P1 pad 26: /P8 -> /B2
- P1 pad 27: /P7 -> /B5
- P1 pad 28: /P6 -> /B7
- P1 pad 29: /P5 -> /B6
- P1 pad 3: /P31 -> unconnected-(P1-Pad3)
- P1 pad 30: /P4 -> /B4
- P1 pad 31: /P3 -> /A7
- P1 pad 32: /P2 -> /A6
- P1 pad 33: /P1 -> /A4
- P1 pad 34: +1V5 -> /A5
- P1 pad 35: /ISP_RST -> /A3
- P1 pad 36: /ISP_SCK -> /A0
- P1 pad 37: /ISP_MOSI -> /A1
- P1 pad 38: /ISP_MISO -> /A2
- P1 pad 4: /P30 -> unconnected-(P1-Pad4)
- P1 pad 5: /P29 -> unconnected-(P1-Pad5)
- P1 pad 6: /P28 -> unconnected-(P1-Pad6)
- P1 pad 7: /P27 -> unconnected-(P1-Pad7)
- P1 pad 8: /P26 -> unconnected-(P1-Pad8)
- P1 pad 9: /P25 -> unconnected-(P1-Pad9)
Routing:
- net /P24: track 90.4 -> 0.00 mm, vias 1 -> 0
- net /P23: track 82.1 -> 0.00 mm, vias 1 -> 0
- net /P4: track 74.6 -> 0.00 mm, vias 1 -> 0
- net /P7: track 66.4 -> 0.00 mm, vias 1 -> 0
- net /P26: track 66.3 -> 0.00 mm, vias 1 -> 0
- net /A6: track 0.00 -> 64.1 mm, vias 0 -> 1
- net /P27: track 60.9 -> 0.00 mm, vias 1 -> 0
- net /A5: track 0.00 -> 56.9 mm, vias 0 -> 1
- net /P25: track 55.6 -> 0.00 mm, vias 1 -> 0
- net /A4: track 0.00 -> 54.9 mm, vias 0 -> 1
- net /P20: track 54.0 -> 0.00 mm, vias 1 -> 0
- net /P3: track 52.7 -> 0.00 mm, vias 1 -> 0
- net /P16: track 50.9 -> 0.00 mm, vias 1 -> 0
- net /P2: track 49.7 -> 0.00 mm, vias 1 -> 0
- net /P19: track 45.7 -> 0.00 mm, vias 1 -> 0
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Other:
- board size 72 x 109 mm -> 72 x 88.2 mm
- copper layers 4 -> 2
- board text added: "A Blueprint Project"
- board text added: "Calcwriter Interface"
- board text added: "Made with <3️ by @Kaemori"
- board text added: "Project: calcwriter.sillyy.gay"
- board text removed: "Logic board here"
- board text removed: "Reference Triad"
