File: calcwriter_pins/calcwriter_pins.kicad_sch (KiCad schematic)
At the start: 35 parts, among them J1 0965-0-15-20-80-14-11-0, J10 0965-0-15-20-80-14-11-0, J11 0965-0-15-20-80-14-11-0, J12 0965-0-15-20-80-14-11-0, J13 0965-0-15-20-80-14-11-0, J14 0965-0-15-20-80-14-11-0, J15 0965-0-15-20-80-14-11-0, J16 0965-0-15-20-80-14-11-0, J17 0965-0-15-20-80-14-11-0, J18 0965-0-15-20-80-14-11-0, J19 0965-0-15-20-80-14-11-0, J2 0965-0-15-20-80-14-11-0, J20 0965-0-15-20-80-14-11-0, J21 0965-0-15-20-80-14-11-0, J22 0965-0-15-20-80-14-11-0, J23 0965-0-15-20-80-14-11-0, J24 0965-0-15-20-80-14-11-0, J25 0965-0-15-20-80-14-11-0, J26 0965-0-15-20-80-14-11-0, J27 0965-0-15-20-80-14-11-0, J28 0965-0-15-20-80-14-11-0, J29 0965-0-15-20-80-14-11-0, J3 0965-0-15-20-80-14-11-0, J30 0965-0-15-20-80-14-11-0, J31 0965-0-15-20-80-14-11-0, J4 0965-0-15-20-80-14-11-0, J5 0965-0-15-20-80-14-11-0, J6 0965-0-15-20-80-14-11-0, J7 0965-0-15-20-80-14-11-0, J8 0965-0-15-20-80-14-11-0, J9 0965-0-15-20-80-14-11-0, P1 FH12-40S-0.5SH_55_

Commit message: did another thing AAAAAAAAAAAAAAAAAAA
Parts:
- removed J10, J11, J12, J13, J14, J15, J16, J17, J18, J19, J20, J21, J22, J23, J24, J25, J26, J27, J28, J29, J3, J30, J31, J5, J6, J7, J8: 0965-0-15-20-80-14-11-0, 0965-0-15-20-80-14-11-0:MILLMAX_0965-0-15-20-80-14-11-0, symbol 0965-0-15-20-80-14-11-0:0965-0-15-20-80-14-11-0
- added A0, A3, A5, A6, A7, B0, B1, B3, B4, B5, B6, B7: 0965-0-15-20-80-14-11-0, pogopin_smd:YZR0156-20033-02, symbol 0965-0-15-20-80-14-11-0:0965-0-15-20-80-14-11-0
- A1: renamed from J1; footprint 0965-0-15-20-80-14-11-0:MILLMAX_0965-0-15-20-80-14-11-0 -> pogopin_smd:YZR0156-20033-02
- A2: renamed from J2; footprint 0965-0-15-20-80-14-11-0:MILLMAX_0965-0-15-20-80-14-11-0 -> pogopin_smd:YZR0156-20033-02
- A4: renamed from J4; footprint 0965-0-15-20-80-14-11-0:MILLMAX_0965-0-15-20-80-14-11-0 -> pogopin_smd:YZR0156-20033-02
- B2: renamed from J9; footprint 0965-0-15-20-80-14-11-0:MILLMAX_0965-0-15-20-80-14-11-0 -> pogopin_smd:YZR0156-20033-02
- CALC_NEG1: renamed from CALC-2; footprint 0965-0-15-20-80-14-11-0:MILLMAX_0965-0-15-20-80-14-11-0 -> pogopin_smd:YZR0156-20033-02
- CALC_POS1: renamed from CALC+2; footprint 0965-0-15-20-80-14-11-0:MILLMAX_0965-0-15-20-80-14-11-0 -> pogopin_smd:YZR0156-20033-02
Connections:
- net P12 is gone; now on net ISP_MISO: P1.22
- net P13 is gone; now on net ISP_MOSI: P1.21
- net P14 is gone; now on net ISP_SCK: P1.20
- net P15 is gone; now on net ISP_RST: P1.19
- net P16 is gone; now on net +1V5: P1.18
- net +1V5: no longer P1.34
- net ISP_MISO: no longer P1.38
- net ISP_MOSI: no longer P1.37
- net ISP_RST: no longer P1.35
- net ISP_SCK: no longer P1.36
- net P1 renamed A1
- net A1: now also P1.37; no longer P1.33
- net P10 renamed B0
- net B0: now also B0.1
- net P11 renamed B3
- net B3: now also B3.1
- net P17: no longer names the net of P1.17
- net P18: no longer names the net of P1.16
- net P19: no longer names the net of P1.15
- net P2 renamed A2
- net A2: now also P1.38; no longer P1.32
- net P20: no longer names the net of P1.14
- net P21: no longer names the net of P1.13
- net P22: no longer names the net of P1.12
- net P23: no longer names the net of P1.11
- net P24: no longer names the net of P1.10
- net P25: no longer names the net of P1.9
- net P26: no longer names the net of P1.8
- net P27: no longer names the net of P1.7
- net P28: no longer names the net of P1.6
- net P29: no longer names the net of P1.5
- net P3 renamed A7
- net A7: now also A7.1
- net P30: no longer names the net of P1.4
- net P31: no longer names the net of P1.3
- net P4 renamed A4
- net A4: now also P1.33; no longer P1.30
- net P5 renamed B6
- net B6: now also B6.1
- net P6 renamed B7
- net B7: now also B7.1
- net P7 renamed B5
- net B5: now also B5.1
- net P8 renamed B2
- net B2: now also B2.1
- net P9 renamed B1
- net B1: now also B1.1; no longer B2.1
- new net A0: A0.1, P1.36
- new net A3: A3.1, P1.35
- new net A5: A5.1, P1.34
- new net A6: A6.1, P1.32
- new net B4: B4.1, P1.30
- no-connect marks 2 -> 17
Other:
- moved on the sheet: A1, A2, A4, B2, CALC_NEG1, CALC_POS1, P1
